File: hardware/4-20ma-wifi.kicad_sch (KiCad schematic)
At the start: 33 parts, among them J1 Screw_Terminal_01x02, J3 Conn_01x19_Female, J5 Conn_01x19_Female, M1 DC-DC_Buck_Step_Module-dc-dc_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, Q2 BSS138, SW1 SW_DIP_x01, U3 ESP32-DEVKITC-32U, U4 LMP8640

Commit message: Minor changes - prepare release
Parts:
- added JP3: SolderJumper_2_Open, Jumper:SolderJumper-2_P1.3mm_Open_Pad1.0x1.5mm, symbol Jumper:SolderJumper_2_Open
- C2: value (none) -> 4.7 uF; footprint (none) -> Capacitor_Tantalum_SMD:CP_EIA-3216-18_Kemet-A
- J2: value (none) -> Screw_Terminal_01x04; footprint (none) -> project_library:TerminalBlock__1x04_P5.00mm_90Degree
- J4: value (none) -> Screw_Terminal_01x03; footprint (none) -> project_library:TerminalBlock__1x03_P5.00mm_90Degree
- JP4: renamed from JP3; value (none) -> SolderJumper_3_Open; footprint (none) -> Jumper:SolderJumper-3_P1.3mm_Open_RoundedPad1.0x1.5mm
- Q1: value (none) -> BSS138; footprint (none) -> Package_TO_SOT_SMD:SOT-23
- U1: value (none) -> LP2980-ADJ; footprint (none) -> Package_TO_SOT_SMD:SOT-23-5
- U2: value (none) -> ADC121C027CIMK; footprint (none) -> Package_TO_SOT_SMD:SOT-23-6
Connections:
- net GND: now also JP3.1 (A); no longer J4.3 (Pin_3), R5.2, U4.4 (-)
- new net: J4.3 (Pin_3), JP3.2 (B), R5.2, U4.4 (-)
Changed lines of the file:
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@@
   (junction (at 82.55 125.73) (diameter 0) (color 0 0 0 0)
   )
-  (junction (at 205.74 50.8) (diameter 0) (color 0 0 0 0)
-  )
   (junction (at 241.3 124.46) (diameter 0) (color 0 0 0 0)
   )
+  (junction (at 205.74 53.34) (diameter 0) (color 0 0 0 0)
+  )
   (junction (at 64.77 81.28) (diameter 0) (color 0 0 0 0)
   )
@@
   (junction (at 58.42 41.91) (diameter 0) (color 0 0 0 0)
   )
-  (junction (at 195.58 44.45) (diameter 0) (color 0 0 0 0)
-  )
   (junction (at 53.34 152.4) (diameter 0) (color 0 0 0 0)
   )
   (junction (at 189.23 44.45) (diameter 0) (color 0 0 0 0)
   )
+  (junction (at 196.85 44.45) (diameter 0) (color 0 0 0 0)
+  )
   (junction (at 99.06 125.73) (diameter 0) (color 0 0 0 0)
   )
@@
     (stroke (width 0) (type default) (color 0 0 0 0))
   )
-  (wire (pts (xy 195.58 44.45) (xy 195.58 50.8))
+  (wire (pts (xy 196.85 52.07) (xy 196.85 53.34))
     (stroke (width 0) (type default) (color 0 0 0 0))
   )
@@
     (stroke (width 0) (type default) (color 0 0 0 0))
   )
-  (wire (pts (xy 195.58 50.8) (xy 205.74 50.8))
-    (stroke (width 0) (type default) (color 0 0 0 0))
-  )
   (wire (pts (xy 63.5 125.73) (xy 63.5 129.54))
     (stroke (width 0) (type default) (color 0 0 0 0))
@@
     (stroke (width 0) (type default) (color 0 0 0 0))
   )
+  (wire (pts (xy 205.74 53.34) (xy 205.74 55.88))
+    (stroke (width 0) (type default) (color 0 0 0 0))
+  )
   (wire (pts (xy 77.47 125.73) (xy 82.55 125.73))
     (stroke (width 0) (type default) (color 0 0 0 0))
@@
     (stroke (width 0) (type default) (color 0 0 0 0))
   )
+  (wire (pts (xy 196.85 53.34) (xy 205.74 53.34))
+    (stroke (width 0) (type default) (color 0 0 0 0))
+  )
   (wire (pts (xy 220.98 50.8) (xy 220.98 55.88))
     (stroke (width 0) (type default) (color 0 0 0 0))
   )
+  (wire (pts (xy 196.85 44.45) (xy 200.66 44.45))
+    (stroke (width 0) (type default) (color 0 0 0 0))
+  )
   (wire (pts (xy 185.42 36.83) (xy 189.23 36.83))
     (stroke (width 0) (type default) (color 0 0 0 0))
@@
     (stroke (width 0) (type default) (color 0 0 0 0))
   )
-  (wire (pts (xy 205.74 50.8) (xy 205.74 55.88))
-    (stroke (width 0) (type default) (color 0 0 0 0))
-  )
   (wire (pts (xy 85.09 88.9) (xy 85.09 90.17))
     (stroke (width 0) (type default) (color 0 0 0 0))
@@
     (stroke (width 0) (type default) (color 0 0 0 0))
   )
-  (wire (pts (xy 195.58 44.45) (xy 200.66 44.45))
-    (stroke (width 0) (type default) (color 0 0 0 0))
-  )
-  (wire (pts (xy 205.74 46.99) (xy 205.74 50.8))
+  (wire (pts (xy 189.23 44.45) (xy 196.85 44.45))
+    (stroke (width 0) (type default) (color 0 0 0 0))
+  )
+  (wire (pts (xy 205.74 46.99) (xy 205.74 53.34))
     (stroke (width 0) (type default) (color 0 0 0 0))
   )
@@
   )
   (wire (pts (xy 200.66 41.91) (xy 200.66 44.45))
-    (stroke (width 0) (type default) (color 0 0 0 0))
-  )
-  (wire (pts (xy 189.23 44.45) (xy 195.58 44.45))
     (stroke (width 0) (type default) (color 0 0 0 0))
   )
@@
       (effects (font (size 1.27 1.27)) (justify left))
     )
-    (property "Value" "" (id 1) (at 44.45 110.49 0)
-      (effects (font (size 1.27 1.27)) (justify left))
-    )
-    (property "Footprint" "" (id 2) (at 64.77 102.87 0)
+    (property "Value" "ADC121C027CIMK" (id 1) (at 44.45 110.49 0)
+      (effects (font (size 1.27 1.27)) (justify left))
+    )
+    (property "Footprint" "Package_TO_SOT_SMD:SOT-23-6" (id 2) (at 64.77 102.87 0)
       (effects (font (size 1.27 1.27)) hide)
     )
@@
       (effects (font (size 1.27 1.27)) (justify left))
     )
-    (property "Value" "" (id 1) (at 88.9 85.7249 0)
-      (effects (font (size 1.27 1.27)) (justify left))
-    )
-    (property "Footprint" "" (id 2) (at 85.09 85.09 0)
+    (property "Value" "4.7 uF" (id 1) (at 88.9 85.7249 0)
+      (effects (font (size 1.27 1.27)) (justify left))
+    )
+    (property "Footprint" "Capacitor_Tantalum_SMD:CP_EIA-3216-18_Kemet-A" (id 2) (at 85.09 85.09 0)
       (effects (font (size 1.27 1.27)) hide)
     )
@@
     (in_bom yes) (on_board yes) (fields_autoplaced)
     (property "Reference" "J4" (id 0) (at 180.34 27.94 0))
-    (property "Value" "" (id 1) (at 180.34 30.48 0))
-    (property "Footprint" "" (id 2) (at 180.34 36.83 0)
+    (property "Value" "Screw_Terminal_01x03" (id 1) (at 180.34 30.48 0))
+    (property "Footprint" "project_library:TerminalBlock__1x03_P5.00mm_90Degree" (id 2) (at 180.34 36.83 0)
       (effects (font (size 1.27 1.27)) hide)
     )
@@
       (effects (font (size 1.27 1.27)) hide)
     )
-    (property "Value" "" (id 1) (at 191.77 19.05 0))
+    (property "Value" "+12V" (id 1) (at 191.77 19.05 0))
     (property "Footprint" "" (id 2) (at 191.77 24.13 0)
       (effects (font (size 1.27 1.27)) hide)
@@
     (in_bom yes) (on_board yes)
     (property "Reference" "J2" (id 0) (at 110.49 135.89 0))
-    (property "Value" "" (id 1) (at 110.49 120.65 0))
-    (property "Footprint" "" (id 2) (at 110.49 147.32 0)
+    (property "Value" "Screw_Terminal_01x04" (id 1) (at 110.49 120.65 0))
+    (property "Footprint" "project_library:TerminalBlock__1x04_P5.00mm_90Degree" (id 2) (at 110.49 147.32 0)
       (effects (font (size 1.27 1.27)) hide)
     )
@@
     (pin "1")
   )
+  (symbol (lib_id "Jumper:SolderJumper_2_Open") (at 196.85 48.26 90) (unit 1)
+    (in_bom yes) (on_board yes) (fields_autoplaced)
+    (property "Reference" "JP3" (id 0) (at 199.39 46.9899 90)
+      (effects (font (size 1.27 1.27)) (justify right))
+    )
+    (property "Value" "SolderJumper_2_Open" (id 1) (at 199.39 49.5299 90)
+      (effects (font (size 1.27 1.27)) (justify right))
+    )
+    (property "Footprint" "Jumper:SolderJumper-2_P1.3mm_Open_Pad1.0x1.5mm" (id 2) (at 196.85 48.26 0)
+      (effects (font (size 1.27 1.27)) hide)
+    )
+    (property "Datasheet" "~" (id 3) (at 196.85 48.26 0)
+      (effects (font (size 1.27 1.27)) hide)
+    )
+    (pin "1")
+    (pin "2")
+  )
   (symbol (lib_id "power:GND") (at 85.09 90.17 0) (unit 1)
     (in_bom yes) (on_board yes)
@@
   (symbol (lib_id "Jumper:SolderJumper_3_Open") (at 228.6 39.37 270) (unit 1)
     (in_bom yes) (on_board yes) (fields_autoplaced)
-    (property "Reference" "JP3" (id 0) (at 231.14 38.0999 90)
-      (effects (font (size 1.27 1.27)) (justify left))
-    )
-    (property "Value" "" (id 1) (at 231.14 40.6399 90)
-      (effects (font (size 1.27 1.27)) (justify left))
-    )
-    (property "Footprint" "" (id 2) (at 228.6 39.37 0)
+    (property "Reference" "JP4" (id 0) (at 231.14 38.0999 90)
+      (effects (font (size 1.27 1.27)) (justify left))
+    )
+    (property "Value" "SolderJumper_3_Open" (id 1) (at 231.14 40.6399 90)
+      (effects (font (size 1.27 1.27)) (justify left))
+    )
+    (property "Footprint" "Jumper:SolderJumper-3_P1.3mm_Open_RoundedPad1.0x1.5mm" (id 2) (at 228.6 39.37 0)
       (effects (font (size 1.27 1.27)) hide)
     )
@@
     (in_bom yes) (on_board yes) (fields_autoplaced)
     (property "Reference" "Q1" (id 0) (at 63.5 142.24 90))
-    (property "Value" "" (id 1) (at 63.5 144.78 90))
-    (property "Footprint" "" (id 2) (at 61.595 139.7 0)
+    (property "Value" "BSS138" (id 1) (at 63.5 144.78 90))
+    (property "Footprint" "Package_TO_SOT_SMD:SOT-23" (id 2) (at 61.595 139.7 0)
       (effects (font (size 1.27 1.27) italic) (justify left) hide)
     )
@@
       (effects (font (size 1.27 1.27)) hide)
     )
-    (property "Value" "" (id 1) (at 58.42 30.48 0))
+    (property "Value" "+12V" (id 1) (at 58.42 30.48 0))
     (property "Footprint" "" (id 2) (at 58.42 35.56 0)
       (effects (font (size 1.27 1.27)) hide)
@@
     (in_bom yes) (on_board yes) (fields_autoplaced)
     (property "Reference" "U1" (id 0) (at 44.45 73.66 0))
-    (property "Value" "" (id 1) (at 44.45 76.2 0))
-    (property "Footprint" "" (id 2) (at 44.45 71.12 0)
+    (property "Value" "LP2980-ADJ" (id 1) (at 44.45 76.2 0))
+    (property "Footprint" "Package_TO_SOT_SMD:SOT-23-5" (id 2) (at 44.45 71.12 0)
       (effects (font (size 1.27 1.27)) hide)
     )
@@
       (reference "JP2") (unit 1) (value "SolderJumper_3_Open") (footprint "Jumper:SolderJumper-3_P1.3mm_Open_RoundedPad1.0x1.5mm")
     )
+    (path "/82851bb1-12a2-41d1-837a-07fd793420e1"
+      (reference "JP3") (unit 1) (value "SolderJumper_2_Open") (footprint "Jumper:SolderJumper-2_P1.3mm_Open_Pad1.0x1.5mm")
+    )
     (path "/a3190785-216c-4699-8169-313b6a5776d8"
-      (reference "JP3") (unit 1) (value "SolderJumper_3_Open") (footprint "Jumper:SolderJumper-3_P1.3mm_Open_RoundedPad1.0x1.5mm")
+      (reference "JP4") (unit 1) (value "SolderJumper_3_Open") (footprint "Jumper:SolderJumper-3_P1.3mm_Open_RoundedPad1.0x1.5mm")
     )
     (path "/de14b838-67aa-4aad-8b9f-4c6183ee4cbd"
